File: ctree.kicad_pcb (KiCad board)
At the start: 2 copper layers, 55 x 55 mm, 52 parts, among them IC1 ATMEGA328P-A, P1 CONN_02X03_PROG, Q1 IRLML6402, Q2 BC817, Q3 IRLML6402, Q4 IRLML6402, SW1 SMD_5.2x5.2, U1 MCP1624

Commit message: Mask settings.
Other:
- rule pad_to_mask_clearance: 0.2 -> 0.05
Changed lines of the file:
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@@
     (links 101)
     (no_connects 1)
-    (area 127.420454 37.420454 182.579546 92.579546)
+    (area 123.5 35 185.000001 96.5)
     (thickness 1.6)
     (drawings 3)
@@
     (pad_size 1.524 1.524)
     (pad_drill 0.762)
-    (pad_to_mask_clearance 0.2)
+    (pad_to_mask_clearance 0.05)
     (aux_axis_origin 126 94)
     (visible_elements 7FFFFFFF)
     (pcbplotparams
-      (layerselection 0x00c30_ffffffff)
+      (layerselection 0x000c0_7ffffffe)
       (usegerberextensions false)
       (excludeedgelayer true)
       (linewidth 0.100000)
       (plotframeref false)
-      (viasonmask false)
+      (viasonmask true)
       (mode 1)
-      (useauxorigin true)
+      (useauxorigin false)
       (hpglpennumber 1)
       (hpglpenspeed 20)
@@
       (padsonsilk false)
       (subtractmaskfromsilk false)
-      (outputformat 1)
-      (mirror false)
+      (outputformat 5)
+      (mirror true)
       (drillshape 0)
       (scaleselection 1)
